File: hardware/pcb/source/TC_IO_REVC.kicad_pcb (KiCad board)
At the start: 2 copper layers, 100 x 100 mm, 78 parts, among them J1 WIRE_PADS_NO_COMPONENT, J10 WIRE_PADS_NO_COMPONENT, J11 WIRE_PADS_NO_COMPONENT, J12 WIRE_PADS_NO_COMPONENT, J13 WIRE_PADS_NO_COMPONENT, J14 WIRE_PADS_NO_COMPONENT, J2 WIRE_PADS_NO_COMPONENT, J3 WIRE_PADS_NO_COMPONENT, J4 WIRE_PADS_NO_COMPONENT, J5 WIRE_PADS_NO_COMPONENT, J6 WIRE_PADS_NO_COMPONENT, J7 WIRE_PADS_NO_COMPONENT, J8 WIRE_PADS_NO_COMPONENT, J9 WIRE_PADS_NO_COMPONENT, U1 MCP3008T-I/SL, U2 SN74HC221DR, U3 SN74HC221DR, U4 SN74HC08DR, U5 SN74HC08DR, U6 SN74HC08DR, U7 MCP100T-300I/TT

Commit message: Replace one-shot ICs with CD74HC221M96 C133954 and refresh review outputs
Parts:
- U2, U3: value SN74HC221DR -> CD74HC221M96
Changed lines of the file:
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@@
 			)
 		)
-		(property "Value" "SN74HC221DR"
+		(property "Value" "CD74HC221M96"
 			(at 0 5.9 0)
 			(layer "F.Fab")
@@
 			)
 		)
-		(property "Value" "SN74HC221DR"
+		(property "Value" "CD74HC221M96"
 			(at 0 5.9 0)
 			(layer "F.Fab")

Commit message: Adopt C2167387 timing capacitors with user accepted approximate timing
Parts:
- C1, C2, C3, C4: value 470nF_5%_X7R_50V -> 470nF_10%_X7R_50V
Changed lines of the file:
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@@
 			)
 		)
-		(property "Value" "470nF_5%_X7R_50V"
+		(property "Value" "470nF_10%_X7R_50V"
 			(at 0 1.85 90)
 			(layer "F.Fab")
@@
 			)
 		)
-		(property "Value" "470nF_5%_X7R_50V"
+		(property "Value" "470nF_10%_X7R_50V"
 			(at 0 1.85 90)
 			(layer "F.Fab")
@@
 			)
 		)
-		(property "Value" "470nF_5%_X7R_50V"
+		(property "Value" "470nF_10%_X7R_50V"
 			(at 0 1.85 90)
 			(layer "F.Fab")
@@
 			)
 		)
-		(property "Value" "470nF_5%_X7R_50V"
+		(property "Value" "470nF_10%_X7R_50V"
 			(at 0 1.85 90)
 			(layer "F.Fab")
